Commit message: adicionado launch file de mapeamento com slam

File: urdf/robovisor_gazebo.xacro (robot description, xacro)
@@ -45,8 +45,8 @@
 				<range>
 					<min>0.3</min>
-					<max>12</max>
+					<max>2</max>
 				</range>
 			</ray>
-			<plugin name="lidar_controller" filename="libgazebo_ros_laser.so">
+			<plugin name="lidar_controller" filename="libgazebo_ros_ray_sensor.so">
 				<ros>
 					<argument>~/out:=scan</argument>

File: urdf/robovisor_joints.xacro (robot description, xacro)
@@ -1,25 +1,35 @@
 <?xml version="1.0"?>
 <robot xmlns:xacro="http://www.ros.org/wiki/xacro" name="robovisor">
+	<joint name="chassis_joint" type="fixed">
+		<parent link="base_link"/>
+		<child link="chassis_link"/>
+		<origin xyz="0 0 ${wheel_radius}" rpy="0 0 0"/>
+	</joint>
+	<joint name="base_footprint_joint" type="fixed">
+        <parent link="base_link"/>
+        <child link="base_footprint"/>
+        <origin xyz="0 0 0" rpy="0 0 0"/>
+    </joint>
 	<joint name="left_wheel_joint" type="continuous">
-		<parent link="base_link"/>
+		<parent link="chassis_link"/>
 		<child link="left_wheel"/>
-		<origin xyz="-${chassis_length/4} ${chassis_width/2} ${wheel_radius}" rpy="-${pi/2} 0 0"/>
+		<origin xyz="-${chassis_length/4} ${chassis_width/2} 0" rpy="-${pi/2} 0 0"/>
 		<axis xyz="0 0 1"/>
 	</joint>
 	<joint name="right_wheel_joint" type="continuous">
-		<parent link="base_link"/>
+		<parent link="chassis_link"/>
 		<child link="right_wheel"/>
-		<origin xyz="-${chassis_length/4} -${chassis_width/2} ${wheel_radius}" rpy="${pi/2} 0 0"/>
+		<origin xyz="-${chassis_length/4} -${chassis_width/2} 0" rpy="${pi/2} 0 0"/>
 		<axis xyz="0 0 -1"/>
 	</joint>
 	<joint name="front_wheel_joint" type="fixed">
-		<parent link="base_link"/>
+		<parent link="chassis_link"/>
 		<child link="front_wheel"/>
-		<origin xyz="${chassis_length/4} 0 ${wheel_radius-chassis_height/2}" rpy="0 0 0"/>
+		<origin xyz="${chassis_length/4} 0 -${chassis_height/2}" rpy="0 0 0"/>
 	</joint>
 	<joint name="lidar_support_joint" type="fixed">
-		<parent link="base_link"/>
+		<parent link="chassis_link"/>
 		<child link="lidar_support"/>
-		<origin xyz="-${chassis_length/4} 0 ${wheel_radius + chassis_height/2 + lidar_length/2}" rpy="0 0 0"/>
+		<origin xyz="-${chassis_length/4} 0 ${chassis_height/2 + lidar_length/2}" rpy="0 0 0"/>
 	</joint>
 	<joint name="lidar_joint" type="fixed">

File: urdf/robovisor_links.xacro (robot description, xacro)
@@ -1,10 +1,12 @@
 <?xml version="1.0"?>
 <robot xmlns:xacro="http://www.ros.org/wiki/xacro" name="robovisor">
-	<link name="base_link">
+	<link name="base_footprint"/>
+	<link name="base_link"/>
+	<link name="chassis_link">
 		<visual>
 			<geometry>
 				<box size="${chassis_length} ${chassis_width} ${chassis_height}"/>
 			</geometry>
-			<origin xyz="0 0 ${wheel_radius}" rpy="0 0 0"/>
+			<origin xyz="0 0 0" rpy="0 0 0"/>
 			<material name="body_color">
 				<color rgba="${body_color}"/>
@@ -15,8 +17,8 @@
 				<box size="${chassis_length} ${chassis_width} ${chassis_height}"/>
 			</geometry>
-			<origin xyz="0 0 ${wheel_radius}" rpy="0 0 0"/>
+			<origin xyz="0 0 0" rpy="0 0 0"/>
 		</collision>
 		<xacro:inertial_box mass="1" x="${chassis_length}" y="${chassis_width}" z="${chassis_height}">
-			<origin xyz="0 0 ${wheel_radius}" rpy="0 0 0"/>
+			<origin xyz="0 0 0" rpy="0 0 0"/>
 		</xacro:inertial_box>
 	</link>
