Commit message: feat: new urdf robot

File: urdf/gazebo/robovisor_gazebo.xacro (robot description, xacro)
@@ -1,23 +1,9 @@
 <?xml version="1.0"?>
 <robot xmlns:xacro="http://www.ros.org/wiki/xacro" name="robovisor">
-	<gazebo reference="chassis">
-		<material>Gazebo/${body_color}</material>
-	</gazebo>
-	<gazebo reference="left_wheel">
-		<material>Gazebo/${wheel_color}</material>
-	</gazebo>
-	<gazebo reference="right_wheel">
-		<material>Gazebo/${wheel_color}</material>
-	</gazebo>
-	<gazebo reference="front_wheel">
-		<material>Gazebo/${wheel_color}</material>
-		<mu1 value="0.001"/>
-		<mu2 value="0.001"/>
-	</gazebo>
 	<gazebo>
 		<plugin name="diff_drive" filename="libgazebo_ros_diff_drive.so">
 			<left_joint>left_wheel_joint</left_joint>
 			<right_joint>right_wheel_joint</right_joint>
-			<wheel_separation>${chassis_width}</wheel_separation>
+			<wheel_separation>${chassis_radius*2 - wheel_length}</wheel_separation>
 			<wheel_diameter>${2*wheel_radius}</wheel_diameter>
 			<max_wheel_torque>200</max_wheel_torque>
@@ -30,5 +16,5 @@
 		</plugin>
 	</gazebo>
-	<gazebo reference="lidar_link">
+	<gazebo reference="laser_link">
 		<sensor name="lidar" type="ray">
 			<pose> 0 0 0 0 0 0 </pose>
@@ -39,6 +25,6 @@
 					<horizontal>
 						<samples>360</samples>
-						<min_angle>-3.14159265</min_angle>
-						<max_angle>3.14159265</max_angle>
+						<min_angle>-${pi/2}</min_angle>
+						<max_angle>${pi/2}</max_angle>
 					</horizontal>
 				</scan>
@@ -57,3 +43,11 @@
 		</sensor>
 	</gazebo>
+	<gazebo reference="caster_n_link">
+		<mu1>0.2</mu1>
+		<mu2>0.2</mu2>
+	</gazebo>
+	<gazebo reference="caster_s_link">
+		<mu1>0.2</mu1>
+		<mu2>0.2</mu2>
+	</gazebo>
 </robot>

File: urdf/includes/robovisor_include.xacro (robot description, xacro)
@@ -1,14 +1,4 @@
 <?xml version="1.0"?>
 <robot xmlns:xacro="http://www.ros.org/wiki/xacro" name="robovisor">
-	<xacro:property name="wheel_radius" value="0.1"/>
-	<xacro:property name="wheel_width" value="0.05"/>
-	<xacro:property name="chassis_length" value="0.4"/>
-	<xacro:property name="chassis_width" value="0.2"/>
-	<xacro:property name="chassis_height" value="0.1"/>
-	<xacro:property name="lidar_radius" value="0.0508"/>
-	<xacro:property name="lidar_length" value="0.055"/>
-	<xacro:property name="camera_length" value="0.015"/>
-	<xacro:property name="camera_width" value="0.13"/>
-	<xacro:property name="camera_heigth" value="0.022"/>
 	<xacro:macro name="inertial_box" params="mass x y z *origin">
 		<inertial>
@@ -38,8 +28,3 @@
 		</inertial>
 	</xacro:macro>
-	<!-- cor das rodas -->
-	<xacro:property name="wheel_color" value="1.0 0.0 0.0 1.0"/>
-	<!-- cor do corpo -->
-	<xacro:property name="body_color" value="0.0 1.0 0.0 1.0"/>
-	<xacro:property name="support_color" value="0.0 0.0 1.0 1.0"/>
 </robot>

File: urdf/robovisor.urdf.xacro (robot description, xacro)
@@ -1,11 +1,16 @@
 <?xml version="1.0"?>
 <robot xmlns:xacro="http://www.ros.org/wiki/xacro" name="robovisor">
-	<!-- header -->
-	<xacro:include filename="robovisor_include.xacro"/>
-	<!-- gazebo macros -->
-	<xacro:include filename="robovisor_gazebo.xacro"/>
-	<!-- links -->
-	<xacro:include filename="robovisor_links.xacro"/>
-	<!-- joints -->
-	<xacro:include filename="robovisor_joints.xacro"/>
+	<!-- includes -->
+	<xacro:include filename="includes/*"/>
+	<!-- gazebo -->
+	<xacro:include filename="gazebo/*"/>
+	<!-- components -->
+	<xacro:include filename="components/*"/>
+	<link name="base_footprint"/>
+	<link name="base_link"/>
+	<joint name="base_footprint_joint" type="fixed">
+		<parent link="base_link"/>
+		<child link="base_footprint"/>
+		<origin xyz="0 0 0" rpy="0 0 0"/>
+	</joint>
 </robot>
