Commit message: fix wheel position

File: urdf/components/robovisor_wheels.xacro (robot description, xacro)
@@ -46,5 +46,5 @@
 		<parent link="right_driver_link"/>
 		<child link="right_wheel_link"/>
-		<origin xyz="0 0 -${driver_length/2}" rpy="0 0 0"/>
+		<origin xyz="0 0 ${driver_length/2}" rpy="0 0 0"/>
 		<axis xyz="0 0 -1"/>
 	</joint>
